File: Audio.kicad_sch (KiCad schematic)
At the start: 15 parts

Commit message: Update Manufacturer/PartNumber accross the whole schema
Signed-off-by: Stefan Agner <stefan@agner.ch>
Parts:
- J?: Manufacturer (none) -> CUI Devices; PartNumber (none) -> SJ2-35954A-SMT-TR
- U?: Manufacturer (none) -> Texas Instruments; PartNumber (none) -> PCM5121PWR
- U?: Manufacturer (none) -> ON Semiconductor; PartNumber (none) -> NCP114AMX330TCG
Changed lines of the file:
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@@
   (junction (at 208.28 39.37) (diameter 0.9144) (color 0 0 0 0))
   (junction (at 210.82 46.99) (diameter 0.9144) (color 0 0 0 0))
+  (no_connect (at 162.56 83.82))
+  (no_connect (at 162.56 86.36))
+  (no_connect (at 162.56 88.9))
   (no_connect (at 162.56 91.44))
-  (no_connect (at 162.56 88.9))
-  (no_connect (at 162.56 86.36))
-  (no_connect (at 162.56 83.82))
   (bus_entry (at 116.84 76.2) (size 2.54 2.54)
     (stroke (width 0.1524) (type solid) (color 0 0 0 0))
@@
   (symbol (lib_id "power:+3.3V") (at 116.84 106.68 90) (unit 1)
     (in_bom yes) (on_board yes)
-    (property "Reference" "#PWR?" (id 0) (at 120.65 106.68 0)
+    (property "Reference" "#PWR0157" (id 0) (at 120.65 106.68 0)
       (effects (font (size 1.27 1.27)) hide)
     )
@@
   (symbol (lib_id "power:+3.3VA") (at 123.19 111.76 90) (unit 1)
     (in_bom yes) (on_board yes)
-    (property "Reference" "#PWR?" (id 0) (at 127 111.76 0)
+    (property "Reference" "#PWR0158" (id 0) (at 127 111.76 0)
       (effects (font (size 1.27 1.27)) hide)
     )
@@
   (symbol (lib_id "power:+3.3V") (at 132.08 39.37 0) (unit 1)
     (in_bom yes) (on_board yes)
-    (property "Reference" "#PWR?" (id 0) (at 132.08 43.18 0)
+    (property "Reference" "#PWR0164" (id 0) (at 132.08 43.18 0)
       (effects (font (size 1.27 1.27)) hide)
     )
@@
   (symbol (lib_id "power:+3.3VA") (at 139.7 66.04 0) (unit 1)
     (in_bom yes) (on_board yes)
-    (property "Reference" "#PWR?" (id 0) (at 139.7 69.85 0)
+    (property "Reference" "#PWR0161" (id 0) (at 139.7 69.85 0)
       (effects (font (size 1.27 1.27)) hide)
     )
@@
   (symbol (lib_id "power:+3.3V") (at 144.78 68.58 0) (unit 1)
     (in_bom yes) (on_board yes)
-    (property "Reference" "#PWR?" (id 0) (at 144.78 72.39 0)
+    (property "Reference" "#PWR0162" (id 0) (at 144.78 72.39 0)
       (effects (font (size 1.27 1.27)) hide)
     )
@@
   (symbol (lib_id "power:+3.3VA") (at 149.86 66.04 0) (unit 1)
     (in_bom yes) (on_board yes)
-    (property "Reference" "#PWR?" (id 0) (at 149.86 69.85 0)
+    (property "Reference" "#PWR0163" (id 0) (at 149.86 69.85 0)
       (effects (font (size 1.27 1.27)) hide)
     )
@@
   (symbol (lib_id "power:+3.3VA") (at 153.67 39.37 0) (unit 1)
     (in_bom yes) (on_board yes)
-    (property "Reference" "#PWR?" (id 0) (at 153.67 43.18 0)
+    (property "Reference" "#PWR0165" (id 0) (at 153.67 43.18 0)
       (effects (font (size 1.27 1.27)) hide)
     )
@@
   (symbol (lib_id "power:+5V") (at 208.28 38.1 0) (unit 1)
     (in_bom yes) (on_board yes)
-    (property "Reference" "#PWR?" (id 0) (at 208.28 41.91 0)
+    (property "Reference" "#PWR0175" (id 0) (at 208.28 41.91 0)
       (effects (font (size 1.27 1.27)) hide)
     )
@@
   (symbol (lib_id "power:+3.3VA") (at 238.76 40.64 270) (unit 1)
     (in_bom yes) (on_board yes)
-    (property "Reference" "#PWR?" (id 0) (at 234.95 40.64 0)
+    (property "Reference" "#PWR0178" (id 0) (at 234.95 40.64 0)
       (effects (font (size 1.27 1.27)) hide)
     )
@@
   (symbol (lib_id "power:+5V") (at 238.76 43.18 270) (unit 1)
     (in_bom yes) (on_board yes)
-    (property "Reference" "#PWR?" (id 0) (at 234.95 43.18 0)
+    (property "Reference" "#PWR0177" (id 0) (at 234.95 43.18 0)
       (effects (font (size 1.27 1.27)) hide)
     )
@@
   (symbol (lib_id "power:GND") (at 123.19 49.53 0) (unit 1)
     (in_bom yes) (on_board yes)
-    (property "Reference" "#PWR?" (id 0) (at 123.19 55.88 0)
+    (property "Reference" "#PWR0166" (id 0) (at 123.19 55.88 0)
       (effects (font (size 1.27 1.27)) hide)
     )
@@
   (symbol (lib_id "power:GND") (at 123.19 104.14 270) (unit 1)
     (in_bom yes) (on_board yes)
-    (property "Reference" "#PWR?" (id 0) (at 116.84 104.14 0)
+    (property "Reference" "#PWR0159" (id 0) (at 116.84 104.14 0)
       (effects (font (size 1.27 1.27)) hide)
     )
@@
   (symbol (lib_id "power:GND") (at 124.46 73.66 180) (unit 1)
     (in_bom yes) (on_board yes)
-    (property "Reference" "#PWR?" (id 0) (at 124.46 67.31 0)
+    (property "Reference" "#PWR0160" (id 0) (at 124.46 67.31 0)
       (effects (font (size 1.27 1.27)) hide)
     )
@@
   (symbol (lib_id "power:GNDA") (at 142.24 121.92 0) (unit 1)
     (in_bom yes) (on_board yes)
-    (property "Reference" "#PWR?" (id 0) (at 142.24 128.27 0)
+    (property "Reference" "#PWR0168" (id 0) (at 142.24 128.27 0)
       (effects (font (size 1.27 1.27)) hide)
     )
@@
   (symbol (lib_id "power:GND") (at 144.78 119.38 0) (unit 1)
     (in_bom yes) (on_board yes)
-    (property "Reference" "#PWR?" (id 0) (at 144.78 125.73 0)
+    (property "Reference" "#PWR0169" (id 0) (at 144.78 125.73 0)
       (effects (font (size 1.27 1.27)) hide)
     )
@@
   (symbol (lib_id "power:GNDA") (at 147.32 121.92 0) (unit 1)
     (in_bom yes) (on_board yes)
-    (property "Reference" "#PWR?" (id 0) (at 147.32 128.27 0)
+    (property "Reference" "#PWR0170" (id 0) (at 147.32 128.27 0)
       (effects (font (size 1.27 1.27)) hide)
     )
@@
   (symbol (lib_id "power:GNDA") (at 166.37 96.52 90) (unit 1)
     (in_bom yes) (on_board yes)
-    (property "Reference" "#PWR?" (id 0) (at 172.72 96.52 0)
+    (property "Reference" "#PWR0171" (id 0) (at 172.72 96.52 0)
       (effects (font (size 1.27 1.27)) hide)
     )
@@
   (symbol (lib_id "power:GNDA") (at 167.64 127 0) (unit 1)
     (in_bom yes) (on_board yes)
-    (property "Reference" "#PWR?" (id 0) (at 167.64 133.35 0)
+    (property "Reference" "#PWR0172" (id 0) (at 167.64 133.35 0)
       (effects (font (size 1.27 1.27)) hide)
     )
@@
   (symbol (lib_id "power:GNDA") (at 171.45 49.53 0) (unit 1)
     (in_bom yes) (on_board yes)
-    (property "Reference" "#PWR?" (id 0) (at 171.45 55.88 0)
+    (property "Reference" "#PWR0174" (id 0) (at 171.45 55.88 0)
       (effects (font (size 1.27 1.27)) hide)
     )
@@
   (symbol (lib_id "power:GNDA") (at 184.15 85.09 0) (unit 1)
     (in_bom yes) (on_board yes)
-    (property "Reference" "#PWR?" (id 0) (at 184.15 91.44 0)
+    (property "Reference" "#PWR0167" (id 0) (at 184.15 91.44 0)
       (effects (font (size 1.27 1.27)) hide)
     )
@@
   (symbol (lib_id "power:GNDA") (at 185.42 111.76 0) (unit 1)
     (in_bom yes) (on_board yes)
-    (property "Reference" "#PWR?" (id 0) (at 185.42 118.11 0)
+    (property "Reference" "#PWR0173" (id 0) (at 185.42 118.11 0)
       (effects (font (size 1.27 1.27)) hide)
     )
@@
   (symbol (lib_id "power:GNDA") (at 210.82 48.26 0) (unit 1)
     (in_bom yes) (on_board yes)
-    (property "Reference" "#PWR?" (id 0) (at 210.82 54.61 0)
+    (property "Reference" "#PWR0176" (id 0) (at 210.82 54.61 0)
       (effects (font (size 1.27 1.27)) hide)
     )
@@
       (effects (font (size 1.27 1.27)) hide)
     )
+    (property "Manufacturer" "CUI Devices" (id 4) (at 193.04 78.74 0)
+      (effects (font (size 1.27 1.27)) hide)
+    )
+    (property "PartNumber" "SJ2-35954A-SMT-TR" (id 5) (at 193.04 78.74 0)
+      (effects (font (size 1.27 1.27)) hide)
+    )
   )
   (symbol (lib_id "custom:NCP114MX") (at 223.52 41.91 0) (unit 1)
@@
       (effects (font (size 1.27 1.27)) hide)
     )
+    (property "Manufacturer" "ON Semiconductor" (id 4) (at 223.52 41.91 0)
+      (effects (font (size 1.27 1.27)) hide)
+    )
+    (property "PartNumber" "NCP114AMX330TCG" (id 5) (at 223.52 41.91 0)
+      (effects (font (size 1.27 1.27)) hide)
+    )
   )
   (symbol (lib_id "Audio:PCM5121PW") (at 144.78 93.98 0) (unit 1)
@@
       (effects (font (size 1.27 1.27)) hide)
     )
+    (property "Manufacturer" "Texas Instruments" (id 4) (at 144.78 93.98 0)
+      (effects (font (size 1.27 1.27)) hide)
+    )
+    (property "PartNumber" "PCM5121PWR" (id 5) (at 144.78 93.98 0)
+      (effects (font (size 1.27 1.27)) hide)
+    )

Commit message: Annotate symbools and assign capacitor footprints
Signed-off-by: Stefan Agner <stefan@agner.ch>
Parts:
- C19, C21, C23, C24, C25, C26, C27: renamed from C?; footprint (none) -> Capacitor_SMD:C_0402_1005Metric
- C20, C22: renamed from C?; footprint (none) -> Capacitor_SMD:C_0805_2012Metric
- gave numbers to parts that had none: 6
Changed lines of the file:
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@@
   (symbol (lib_id "Device:R_Small") (at 144.78 48.26 270) (unit 1)
     (in_bom yes) (on_board yes)
-    (property "Reference" "R?" (id 0) (at 144.78 46.3488 90))
+    (property "Reference" "R15" (id 0) (at 144.78 46.3488 90))
     (property "Value" "0R" (id 1) (at 144.78 50.908 90))
     (property "Footprint" "" (id 2) (at 144.78 48.26 0)
@@
   (symbol (lib_id "Device:R_Small") (at 175.26 76.2 90) (unit 1)
     (in_bom yes) (on_board yes)
-    (property "Reference" "R?" (id 0) (at 175.26 71.12 90))
+    (property "Reference" "R16" (id 0) (at 175.26 71.12 90))
     (property "Value" "470R" (id 1) (at 175.26 73.66 90))
     (property "Footprint" "" (id 2) (at 175.26 76.2 0)
@@
   (symbol (lib_id "Device:R_Small") (at 175.26 78.74 90) (unit 1)
     (in_bom yes) (on_board yes)
-    (property "Reference" "R?" (id 0) (at 175.26 83.82 90))
+    (property "Reference" "R17" (id 0) (at 175.26 83.82 90))
     (property "Value" "470R" (id 1) (at 175.26 81.28 90))
     (property "Footprint" "" (id 2) (at 175.26 78.74 0)
@@
   (symbol (lib_id "Device:C_Small") (at 123.19 44.45 0) (unit 1)
     (in_bom yes) (on_board yes)
-    (property "Reference" "C?" (id 0) (at 125.73 43.18 0)
+    (property "Reference" "C19" (id 0) (at 125.73 43.18 0)
       (effects (font (size 1.27 1.27)) (justify left))
     )
@@
       (effects (font (size 1.27 1.27)) (justify left))
     )
-    (property "Footprint" "" (id 2) (at 123.19 44.45 0)
+    (property "Footprint" "Capacitor_SMD:C_0402_1005Metric" (id 2) (at 123.19 44.45 0)
       (effects (font (size 1.27 1.27)) hide)
     )
@@
   (symbol (lib_id "Device:C_Small") (at 132.08 44.45 0) (unit 1)
     (in_bom yes) (on_board yes)
-    (property "Reference" "C?" (id 0) (at 134.62 43.18 0)
+    (property "Reference" "C20" (id 0) (at 134.62 43.18 0)
       (effects (font (size 1.27 1.27)) (justify left))
     )
@@
       (effects (font (size 1.27 1.27)) (justify left))
     )
-    (property "Footprint" "" (id 2) (at 132.08 44.45 0)
+    (property "Footprint" "Capacitor_SMD:C_0805_2012Metric" (id 2) (at 132.08 44.45 0)
       (effects (font (size 1.27 1.27)) hide)
     )
@@
   (symbol (lib_id "Device:C_Small") (at 153.67 44.45 0) (unit 1)
     (in_bom yes) (on_board yes)
-    (property "Reference" "C?" (id 0) (at 156.21 43.18 0)
+    (property "Reference" "C21" (id 0) (at 156.21 43.18 0)
       (effects (font (size 1.27 1.27)) (justify left))
     )
@@
       (effects (font (size 1.27 1.27)) (justify left))
     )
-    (property "Footprint" "" (id 2) (at 153.67 44.45 0)
+    (property "Footprint" "Capacitor_SMD:C_0402_1005Metric" (id 2) (at 153.67 44.45 0)
       (effects (font (size 1.27 1.27)) hide)
     )
@@
   (symbol (lib_id "Device:C_Small") (at 163.83 44.45 0) (unit 1)
     (in_bom yes) (on_board yes)
-    (property "Reference" "C?" (id 0) (at 166.37 43.18 0)
+    (property "Reference" "C22" (id 0) (at 166.37 43.18 0)
       (effects (font (size 1.27 1.27)) (justify left))
     )
@@
       (effects (font (size 1.27 1.27)) (justify left))
     )
-    (property "Footprint" "" (id 2) (at 163.83 44.45 0)
+    (property "Footprint" "Capacitor_SMD:C_0805_2012Metric" (id 2) (at 163.83 44.45 0)
       (effects (font (size 1.27 1.27)) hide)
     )
@@
   (symbol (lib_id "Device:C_Small") (at 167.64 121.92 0) (mirror y) (unit 1)
     (in_bom yes) (on_board yes)
-    (property "Reference" "C?" (id 0) (at 170.18 120.65 0)
+    (property "Reference" "C23" (id 0) (at 170.18 120.65 0)
       (effects (font (size 1.27 1.27)) (justify right))
     )
@@
       (effects (font (size 1.27 1.27)) (justify right))
     )
-    (property "Footprint" "" (id 2) (at 167.64 121.92 0)
+    (property "Footprint" "Capacitor_SMD:C_0402_1005Metric" (id 2) (at 167.64 121.92 0)
       (effects (font (size 1.27 1.27)) hide)
     )
@@
   (symbol (lib_id "Device:C_Small") (at 170.18 102.87 0) (unit 1)
     (in_bom yes) (on_board yes)
-    (property "Reference" "C?" (id 0) (at 172.72 101.6 0)
+    (property "Reference" "C24" (id 0) (at 172.72 101.6 0)
       (effects (font (size 1.27 1.27)) (justify left))
     )
@@
       (effects (font (size 1.27 1.27)) (justify left))
     )
-    (property "Footprint" "" (id 2) (at 170.18 102.87 0)
+    (property "Footprint" "Capacitor_SMD:C_0402_1005Metric" (id 2) (at 170.18 102.87 0)
       (effects (font (size 1.27 1.27)) hide)
     )
@@
   (symbol (lib_id "Device:C_Small") (at 171.45 44.45 0) (unit 1)
     (in_bom yes) (on_board yes)
-    (property "Reference" "C?" (id 0) (at 173.99 43.18 0)
+    (property "Reference" "C25" (id 0) (at 173.99 43.18 0)
       (effects (font (size 1.27 1.27)) (justify left))
     )
@@
       (effects (font (size 1.27 1.27)) (justify left))
     )
-    (property "Footprint" "" (id 2) (at 171.45 44.45 0)
+    (property "Footprint" "Capacitor_SMD:C_0402_1005Metric" (id 2) (at 171.45 44.45 0)
       (effects (font (size 1.27 1.27)) hide)
     )
@@
   (symbol (lib_id "Device:C_Small") (at 176.53 109.22 270) (unit 1)
     (in_bom yes) (on_board yes)
-    (property "Reference" "C?" (id 0) (at 176.53 115.57 90))
+    (property "Reference" "C26" (id 0) (at 176.53 115.57 90))
     (property "Value" "100n" (id 1) (at 176.53 113.03 90))
-    (property "Footprint" "" (id 2) (at 176.53 109.22 0)
+    (property "Footprint" "Capacitor_SMD:C_0402_1005Metric" (id 2) (at 176.53 109.22 0)
       (effects (font (size 1.27 1.27)) hide)
     )
@@
   (symbol (lib_id "Device:C_Small") (at 204.47 43.18 0) (unit 1)
     (in_bom yes) (on_board yes)
-    (property "Reference" "C?" (id 0) (at 207.01 41.91 0)
+    (property "Reference" "C27" (id 0) (at 207.01 41.91 0)
       (effects (font (size 1.27 1.27)) (justify left))
     )
@@
       (effects (font (size 1.27 1.27)) (justify left))
     )
-    (property "Footprint" "" (id 2) (at 204.47 43.18 0)
+    (property "Footprint" "Capacitor_SMD:C_0402_1005Metric" (id 2) (at 204.47 43.18 0)
       (effects (font (size 1.27 1.27)) hide)
     )
@@
   (symbol (lib_id "Connector:AudioJack3") (at 193.04 78.74 180) (unit 1)
     (in_bom yes) (on_board yes)
-    (property "Reference" "J?" (id 0) (at 200.1521 77.0064 0)
+    (property "Reference" "J8" (id 0) (at 200.1521 77.0064 0)
       (effects (font (size 1.27 1.27)) (justify right))
     )
@@
   (symbol (lib_id "custom:NCP114MX") (at 223.52 41.91 0) (unit 1)
     (in_bom yes) (on_board yes)
-    (property "Reference" "U?" (id 0) (at 223.52 35.0582 0))
+    (property "Reference" "U11" (id 0) (at 223.52 35.0582 0))
     (property "Value" "NCP114AMX330TCG" (id 1) (at 223.52 37.3569 0))
     (property "Footprint" "" (id 2) (at 223.52 41.91 0)
@@
   (symbol (lib_id "Audio:PCM5121PW") (at 144.78 93.98 0) (unit 1)
     (in_bom yes) (on_board yes)
-    (property "Reference" "U?" (id 0) (at 130.81 72.39 0))
+    (property "Reference" "U10" (id 0) (at 130.81 72.39 0))
     (property "Value" "PCM5121PW" (id 1) (at 154.94 72.39 0))
     (property "Footprint" "Package_SO:TSSOP-28_4.4x9.7mm_P0.65mm" (id 2) (at 144.78 93.98 0)
