File: Ethernet.kicad_sch (KiCad schematic)
At the start: 8 parts, among them J9 RJ45_LINK-PP_LPJG0926HENL_Hor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, U12 TPD4EUSB30, U13 TPD4EUSB30

Commit message: Define footprint for remaining parts
- Fix footprint for 02x05 pin header
- Add footprint for Bourns SDR1006 Inductor (PoE)
- Define footprints for inductors
- Define footprints for ferrite beads
- Define footprint for fuse
- Define footprints for all resistors
- Define footprints for SD card and other components
- Switch ON Semi NCP114MX with TI TLV73333PDBV

Signed-off-by: Stefan Agner <stefan@agner.ch>
Parts:
- R18, R19, R20: footprint (none) -> Resistor_SMD:R_0402_1005Metric
Changed lines of the file:
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@@
     (comment 2 "Light Blue")
   )
+  (bus_alias "ETH" (members "TD1+" "TD1-" "TD2+" "TD2-" "TD3+" "TD3-" "TD4+" "TD4-" "LED_YELLOW" "LED_GREEN"))
   (bus_alias "PoE" (members "VC1" "VC2" "VC3" "VC4"))
-  (bus_alias "ETH" (members "TD1+" "TD1-" "TD2+" "TD2-" "TD3+" "TD3-" "TD4+" "TD4-" "LED_YELLOW" "LED_GREEN"))
   (junction (at 153.67 80.01) (diameter 0.9144) (color 0 0 0 0))
   (junction (at 177.8 130.81) (diameter 0.9144) (color 0 0 0 0))
@@
     (property "Reference" "R18" (id 0) (at 148.59 50.8 90))
     (property "Value" "470Ω" (id 1) (at 148.59 53.34 90))
-    (property "Footprint" "" (id 2) (at 148.59 55.88 0)
+    (property "Footprint" "Resistor_SMD:R_0402_1005Metric" (id 2) (at 148.59 55.88 0)
       (effects (font (size 1.27 1.27)) hide)
     )
@@
     (property "Reference" "R19" (id 0) (at 146.05 121.92 90))
     (property "Value" "470Ω" (id 1) (at 151.13 121.92 90))
-    (property "Footprint" "" (id 2) (at 148.59 119.38 0)
+    (property "Footprint" "Resistor_SMD:R_0402_1005Metric" (id 2) (at 148.59 119.38 0)
       (effects (font (size 1.27 1.27)) hide)
     )
@@
     (property "Reference" "R20" (id 0) (at 181.7432 133.35 0))
     (property "Value" "0R" (id 1) (at 190.392 135.89 0))
-    (property "Footprint" "" (id 2) (at 184.15 135.89 0)
-      (effects (font (size 1.27 1.27)) hide)
-    )
+    (property "Footprint" "Resistor_SMD:R_0402_1005Metric" (id 2) (at 184.15 135.89 0)
+      (effects (font (size 1.27 1.27)) hide)
+    )
