File: sdcard.kicad_sch (KiCad schematic)
At the start: 4 parts, among them J12 Micro_SD_Card_Det, U19 RT9742GGJ5

Commit message: Define footprint for remaining parts
- Fix footprint for 02x05 pin header
- Add footprint for Bourns SDR1006 Inductor (PoE)
- Define footprints for inductors
- Define footprints for ferrite beads
- Define footprint for fuse
- Define footprints for all resistors
- Define footprints for SD card and other components
- Switch ON Semi NCP114MX with TI TLV73333PDBV

Signed-off-by: Stefan Agner <stefan@agner.ch>
Parts:
- J12: Manufacturer (none) -> Molex; PartNumber (none) -> 104031-0811
- R36: footprint (none) -> Resistor_SMD:R_0402_1005Metric
Changed lines of the file:
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@@
     (property "Reference" "R36" (id 0) (at 66.675 85.725 90))
     (property "Value" "10k" (id 1) (at 70.485 85.725 90))
-    (property "Footprint" "" (id 2) (at 69.215 83.185 0)
+    (property "Footprint" "Resistor_SMD:R_0402_1005Metric" (id 2) (at 69.215 83.185 0)
       (effects (font (size 1.27 1.27)) hide)
     )
@@
     )
     (property "Config" "+SDCard" (id 4) (at 103.505 50.165 0))
+    (property "Manufacturer" "Molex" (id 4) (at 102.235 70.485 0)
+      (effects (font (size 1.27 1.27)) hide)
+    )
+    (property "PartNumber" "104031-0811" (id 5) (at 102.235 70.485 0)
+      (effects (font (size 1.27 1.27)) hide)
+    )
   )
 )
