File: Amber.kicad_sch (KiCad schematic)
At the start: 15 parts

Commit message: Renmae LightBlue to Amber
Signed-off-by: Stefan Agner <stefan@agner.ch>
Parts:
- H5, H6: footprint LightBlue:DrillSlot_Plated_3.5x2.5mm -> Amber:DrillSlot_Plated_3.5x2.5mm
- HS1: footprint LightBlue:Heatsink_56x56mm_2xFixation3.2mm -> Amber:Heatsink_56x56mm_2xFixation3.2mm
Changed lines of the file:
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@@
     (company "Nabu Casa")
     (comment 1 "www.nabucasa.com")
-    (comment 2 "Light Blue")
+    (comment 2 "Amber")
   )
   (wire (pts (xy 59.69 44.45) (xy 90.17 44.45))
@@
       (effects (font (size 1.27 1.27)) (justify left))
     )
-    (property "Footprint" "LightBlue:DrillSlot_Plated_3.5x2.5mm" (id 2) (at 111.76 182.88 0)
+    (property "Footprint" "Amber:DrillSlot_Plated_3.5x2.5mm" (id 2) (at 111.76 182.88 0)
       (effects (font (size 1.27 1.27)) hide)
     )
@@
       (effects (font (size 1.27 1.27)) (justify left))
     )
-    (property "Footprint" "LightBlue:DrillSlot_Plated_3.5x2.5mm" (id 2) (at 111.76 190.5 0)
+    (property "Footprint" "Amber:DrillSlot_Plated_3.5x2.5mm" (id 2) (at 111.76 190.5 0)
       (effects (font (size 1.27 1.27)) hide)
     )
@@
       (effects (font (size 1.27 1.27)) (justify left))
     )
-    (property "Footprint" "LightBlue:Heatsink_56x56mm_2xFixation3.2mm" (id 2) (at 133.6548 185.42 0)
+    (property "Footprint" "Amber:Heatsink_56x56mm_2xFixation3.2mm" (id 2) (at 133.6548 185.42 0)
       (effects (font (size 1.27 1.27)) hide)
     )
@@
     )
     (path "/37de04fb-2d22-493d-a648-e024c9d5a4fc"
-      (reference "H5") (unit 1) (value "MountingHole") (footprint "LightBlue:DrillSlot_Plated_3.5x2.5mm")
+      (reference "H5") (unit 1) (value "MountingHole") (footprint "Amber:DrillSlot_Plated_3.5x2.5mm")
     )
     (path "/bfcec0b4-32c4-4ebf-8bb4-4766287797f1"
-      (reference "H6") (unit 1) (value "MountingHole") (footprint "LightBlue:DrillSlot_Plated_3.5x2.5mm")
+      (reference "H6") (unit 1) (value "MountingHole") (footprint "Amber:DrillSlot_Plated_3.5x2.5mm")
     )
     (path "/cd73f910-31d6-4226-a110-18f09eef8514"
-      (reference "HS1") (unit 1) (value "Heatsink") (footprint "LightBlue:Heatsink_56x56mm_2xFixation3.2mm")
+      (reference "HS1") (unit 1) (value "Heatsink") (footprint "Amber:Heatsink_56x56mm_2xFixation3.2mm")
     )
     (path "/c7bf4e1f-6bd1-4be7-9e56-1bd438bf5d42/eda8ae3b-dbdd-4e73-8dc6-e01177bfb4f7"
-      (reference "J1") (unit 1) (value "Barrel_Jack") (footprint "LightBlue:BarrelJack_CUI_PJ-002A")
+      (reference "J1") (unit 1) (value "Barrel_Jack") (footprint "Amber:BarrelJack_CUI_PJ-002A")
     )
     (path "/18c18357-12fa-4472-a108-e954e5bd7840/6dd5e861-e5d4-4759-b127-4958e3f04beb"
-      (reference "J2") (unit 1) (value "RJ45_LINK-PP_LPJG0926HENL_Horizontal") (footprint "LightBlue:RJ45_LINK-PP_LPJG0926HENL_Horizontal")
+      (reference "J2") (unit 1) (value "RJ45_LINK-PP_LPJG0926HENL_Horizontal") (footprint "Amber:RJ45_LINK-PP_LPJG0926HENL_Horizontal")
     )
     (path "/aa1d8d83-5167-420c-9ee7-3e4dcc942bfc/e0469852-771a-434b-963a-8ecb4c38b617"
@@
     )
     (path "/a9e0a5b9-8f0f-46f3-b2b0-a429c678afed/45c3bea5-38ff-4276-ad09-4c18c95d656c"
-      (reference "J5") (unit 1) (value "AudioJack") (footprint "LightBlue:Jack_3.5mm_XKB_PJ-3270_Horizontal")
+      (reference "J5") (unit 1) (value "AudioJack") (footprint "Amber:Jack_3.5mm_XKB_PJ-3270_Horizontal")
     )
     (path "/7c248bd3-8232-4777-a40c-eab53460cf85/fe81f5fa-e1ac-4968-a654-7214906ce5ba"
@@
     )
     (path "/a1a835e0-c072-4609-9cb4-4b95bf746f54/1247548e-da2d-4da5-8e9d-cdb0bd0eeb39"
-      (reference "J12") (unit 1) (value "Bus_M.2_Socket_M") (footprint "LightBlue:TE_1-2199230-3_Bus_M.2_M_H4.2mm_P0.5mm_2280_Horizontal")
+      (reference "J12") (unit 1) (value "Bus_M.2_Socket_M") (footprint "Amber:TE_1-2199230-3_Bus_M.2_M_H4.2mm_P0.5mm_2280_Horizontal")
     )
     (path "/6888556d-e390-44b5-977e-8a0092745a4b/d2f558fb-acd9-4c71-93bb-37883bf1acff"
@@
     )
     (path "/6888556d-e390-44b5-977e-8a0092745a4b/8e4bf553-ed00-4225-96a1-870ada5deeea"
-      (reference "Q2") (unit 1) (value "BSZ440N10NS3GATMA1") (footprint "LightBlue:PG-TSDSON-8")
+      (reference "Q2") (unit 1) (value "BSZ440N10NS3GATMA1") (footprint "Amber:PG-TSDSON-8")
     )
     (path "/7c248bd3-8232-4777-a40c-eab53460cf85/f65f5283-bc09-4a32-875e-7aff6fe23fca"
@@
     )
     (path "/6888556d-e390-44b5-977e-8a0092745a4b/897f43a2-d08b-4609-bc6b-c864c929a423"
-      (reference "T1") (unit 1) (value "PA2467NL") (footprint "LightBlue:Transformer_Pulse_PA2467NL")
+      (reference "T1") (unit 1) (value "PA2467NL") (footprint "Amber:Transformer_Pulse_PA2467NL")
     )
     (path "/7c248bd3-8232-4777-a40c-eab53460cf85/b88488bf-0e8e-4b66-85b8-98e34521bccf"
@@
     )
     (path "/7c248bd3-8232-4777-a40c-eab53460cf85/b131b144-fc54-40cc-8411-449b069a57ca"
-      (reference "U1") (unit 1) (value "RaspberryPi-CM4Lite") (footprint "LightBlue:RaspberryPi-CM4")
+      (reference "U1") (unit 1) (value "RaspberryPi-CM4Lite") (footprint "Amber:RaspberryPi-CM4")
     )
     (path "/7c248bd3-8232-4777-a40c-eab53460cf85/e774090e-475c-4e3f-aa6e-6c912d7ab3b3"
-      (reference "U1") (unit 2) (value "RaspberryPi-CM4Lite") (footprint "LightBlue:RaspberryPi-CM4")
+      (reference "U1") (unit 2) (value "RaspberryPi-CM4Lite") (footprint "Amber:RaspberryPi-CM4")
     )
     (path "/7c248bd3-8232-4777-a40c-eab53460cf85/4dd6bcbf-26fd-4425-8fa4-2095d8aa465e"
-      (reference "U2") (unit 1) (value "DF40C-100DS-0.4V") (footprint "LightBlue:Hirose_DF40_DF40C-100DS-0.4V_2x50_P0.40mm_Vertical_Virtual")
+      (reference "U2") (unit 1) (value "DF40C-100DS-0.4V") (footprint "Amber:Hirose_DF40_DF40C-100DS-0.4V_2x50_P0.40mm_Vertical_Virtual")
     )
     (path "/7c248bd3-8232-4777-a40c-eab53460cf85/736345e1-e2da-4fe0-b090-447995db5e70"
-      (reference "U3") (unit 1) (value "DF40C-100DS-0.4V") (footprint "LightBlue:Hirose_DF40_DF40C-100DS-0.4V_2x50_P0.40mm_Vertical_Virtual")
+      (reference "U3") (unit 1) (value "DF40C-100DS-0.4V") (footprint "Amber:Hirose_DF40_DF40C-100DS-0.4V_2x50_P0.40mm_Vertical_Virtual")
     )
     (path "/aa1d8d83-5167-420c-9ee7-3e4dcc942bfc/15a1c1c3-ed5e-4bb3-a60a-04e93ff6b7c2"
@@
     )
     (path "/12f6ca59-5dee-4aea-b4bb-e4b9cab2885b/c09bd077-0d29-41a3-91d8-7b26a3246dec"
-      (reference "U11") (unit 1) (value "SiliconLabs-MGM210P") (footprint "LightBlue:SiliconLabs_MGM210P")
+      (reference "U11") (unit 1) (value "SiliconLabs-MGM210P") (footprint "Amber:SiliconLabs_MGM210P")
     )
     (path "/a9e0a5b9-8f0f-46f3-b2b0-a429c678afed/1e9ebda2-59cb-4701-873a-d55dee03ba02"
@@
     )
     (path "/6888556d-e390-44b5-977e-8a0092745a4b/1ac452f1-c834-435c-b0e7-9e1426e4cc85"
-      (reference "U23") (unit 1) (value "TPS23734") (footprint "LightBlue:Texas_VQFN-47-2EP_5x7mm_P0.4mm_ThermalVias")
+      (reference "U23") (unit 1) (value "TPS23734") (footprint "Amber:Texas_VQFN-47-2EP_5x7mm_P0.4mm_ThermalVias")
     )
     (path "/6888556d-e390-44b5-977e-8a0092745a4b/facccdfa-9875-4bdc-aa78-dfb84f69ada3"

Commit message: Fix/improve various parts
- U7: Define Manufacturer/PartNumber
- J13: Define Manufacturer/PartNumber
- L2: Fix PartNumber (remove unprintable characters)
- C85: Change to our preferred supplier Nichicon
- J9: DNP (not used by default, avoid potential issues with FCC approval)
- Y1/Y2: Define frequency and load capacitance in value
- JP1: Use sensible part value
- C106: Fix Config field
- Remove heat sink and CM4 from BOM (handled in product assembly BOM)

Signed-off-by: Stefan Agner <stefan@agner.ch>
Parts:
- HS1: now left out of the parts list
Changed lines of the file:
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@@
   )
   (symbol (lib_id "Mechanical:Heatsink") (at 133.35 185.42 0) (unit 1)
-    (in_bom yes) (on_board yes)
+    (in_bom no) (on_board yes)
     (property "Reference" "HS1" (id 0) (at 136.9569 182.3656 0)
       (effects (font (size 1.27 1.27)) (justify left))
@@
     )
     (path "/aa1d8d83-5167-420c-9ee7-3e4dcc942bfc/21f085b4-1176-4778-97ba-f2d2acc22e65"
-      (reference "JP1") (unit 1) (value "JP_USB_DEVICE_SEL") (footprint "Connector_PinHeader_2.54mm:PinHeader_1x03_P2.54mm_Vertical")
+      (reference "JP1") (unit 1) (value "Conn_01x03_Male") (footprint "Connector_PinHeader_2.54mm:PinHeader_1x03_P2.54mm_Vertical")
     )
     (path "/7c248bd3-8232-4777-a40c-eab53460cf85/e968abf9-4624-4f9a-a426-43f6f969f7bc"
@@
     )
     (path "/aa1d8d83-5167-420c-9ee7-3e4dcc942bfc/fbf0dbc2-bf7a-418f-bca2-8248332c89a0"
-      (reference "Y1") (unit 1) (value "12MHz") (footprint "Crystal:Crystal_SMD_3225-4Pin_3.2x2.5mm")
+      (reference "Y1") (unit 1) (value "12MHz{slash}10pF") (footprint "Crystal:Crystal_SMD_3225-4Pin_3.2x2.5mm")
     )
     (path "/441a9908-1e74-440b-b462-bdf6815583fe/df3c69bc-5fed-486a-8538-f634d169db1f"
-      (reference "Y2") (unit 1) (value "X32K768S301") (footprint "Crystal:Crystal_SMD_3215-2Pin_3.2x1.5mm")
+      (reference "Y2") (unit 1) (value "32768Hz{slash}12.5pF") (footprint "Crystal:Crystal_SMD_3215-2Pin_3.2x1.5mm")
     )
   )
