File: PoE.kicad_sch (KiCad schematic)
At the start: 80 parts, among them J13 Conn_01x03_Male, Q2 BSZ440N10NS3GATMA1, Q3 MMBTA06, T1 PA2467NL, U23 MP8008, U24 TCMT1107, U28 TCMT1107, U29 TL431DBZ

Commit message: Rename Amber to Yellow everywhere
Signed-off-by: Stefan Agner <stefan@agner.ch>
Parts:
- FL1: footprint Amber:L_CommonModeChoke_Murata_DLW5B -> Yellow:L_CommonModeChoke_Murata_DLW5B; symbol Amber:Filter_EMI_LL_1243 -> Yellow:Filter_EMI_LL_1243
- Q2: footprint Amber:PG-TSDSON-8 -> Yellow:PG-TSDSON-8
- T1: footprint Amber:Transformer_Pulse_PA2467NL -> Yellow:Transformer_Pulse_PA2467NL; symbol Amber:Transformer_Pulse_PA2476NL -> Yellow:Transformer_Pulse_PA2476NL
- U23: symbol Amber:MP8008 -> Yellow:MP8008
Changed lines of the file:
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@@
     (pin "2")
   )
-  (symbol (lib_id "Amber:Filter_EMI_LL_1243") (at 73.66 69.85 0) (unit 1)
+  (symbol (lib_id "Yellow:Filter_EMI_LL_1243") (at 73.66 69.85 0) (unit 1)
     (in_bom yes) (on_board yes)
     (property "Reference" "FL1" (id 0) (at 73.66 62.23 0))
     (property "Value" "1k@100MHz{slash}500mA" (id 1) (at 73.66 64.135 0))
-    (property "Footprint" "Amber:L_CommonModeChoke_Murata_DLW5B" (id 2) (at 73.66 68.834 0)
+    (property "Footprint" "Yellow:L_CommonModeChoke_Murata_DLW5B" (id 2) (at 73.66 68.834 0)
       (effects (font (size 1.27 1.27)) hide)
     )
@@
     (pin "2")
   )
-  (symbol (lib_id "Amber:Transformer_Pulse_PA2476NL") (at 199.39 45.72 0) (unit 1)
+  (symbol (lib_id "Yellow:Transformer_Pulse_PA2476NL") (at 199.39 45.72 0) (unit 1)
     (in_bom yes) (on_board yes) (fields_autoplaced)
     (property "Reference" "T1" (id 0) (at 199.39 27.94 0))
     (property "Value" "PA2467NL" (id 1) (at 199.39 30.48 0))
-    (property "Footprint" "Amber:Transformer_Pulse_PA2467NL" (id 2) (at 199.39 45.72 0)
+    (property "Footprint" "Yellow:Transformer_Pulse_PA2467NL" (id 2) (at 199.39 45.72 0)
       (effects (font (size 1.27 1.27)) hide)
     )
@@
       (effects (font (size 1.27 1.27)) (justify left))
     )
-    (property "Footprint" "Amber:PG-TSDSON-8" (id 2) (at 177.8 111.125 0)
+    (property "Footprint" "Yellow:PG-TSDSON-8" (id 2) (at 177.8 111.125 0)
       (effects (font (size 1.27 1.27) italic) (justify left) hide)
     )
@@
     (pin "4")
   )
-  (symbol (lib_id "Amber:MP8008") (at 90.17 130.81 0) (unit 1)
+  (symbol (lib_id "Yellow:MP8008") (at 90.17 130.81 0) (unit 1)
     (in_bom yes) (on_board yes)
     (property "Reference" "U23" (id 0) (at 78.105 106.68 0))
